File: Hardware/arduino-nano-dcc-v2.brd (EAGLE design)
At the start: 58.7 x 44.5 mm, 45 parts, among them IC1 7805TV, IC3 MEGA328-P, Q2 TIP41C, X1 22-23-2031

Commit message: Added values to components and added partlist.
Parts:
- C1, C2: value (none) -> 33pF
- C4, C6, C7: value (none) -> 100n
- Q1: value (none) -> 16MHz
Changed lines of the file:
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@@
 <attribute name="VALUE" x="10.795" y="24.14" size="1.778" layer="27" ratio="10"/>
 </element>
-<element name="Q1" library="crystal" library_urn="urn:adsk.eagle:library:204" package="HC49U-V" package3d_urn="urn:adsk.eagle:package:12075/1" value="" x="31.75" y="13.345" smashed="yes" rot="R90">
+<element name="Q1" library="crystal" library_urn="urn:adsk.eagle:library:204" package="HC49U-V" package3d_urn="urn:adsk.eagle:package:12075/1" value="16MHz" x="31.75" y="13.345" smashed="yes" rot="R90">
 <attribute name="MF" value="" x="31.75" y="13.345" size="1.778" layer="27" rot="R90" display="off"/>
 <attribute name="MPN" value="" x="31.75" y="13.345" size="1.778" layer="27" rot="R90" display="off"/>
@@
 <attribute name="VALUE" x="35.941" y="8.265" size="1.27" layer="27" ratio="10" rot="R90"/>
 </element>
-<element name="C1" library="rcl" library_urn="urn:adsk.eagle:library:334" package="C025-024X044" package3d_urn="urn:adsk.eagle:package:23630/1" value="" x="33.02" y="5.725" smashed="yes" rot="R270">
+<element name="C1" library="rcl" library_urn="urn:adsk.eagle:library:334" package="C025-024X044" package3d_urn="urn:adsk.eagle:package:23630/1" value="33pF" x="33.02" y="5.725" smashed="yes" rot="R270">
 <attribute name="NAME" x="34.417" y="7.503" size="1.27" layer="25" ratio="10" rot="R270"/>
 <attribute name="POPULARITY" value="56" x="33.02" y="5.725" size="1.778" layer="27" rot="R270" display="off"/>
@@
 <attribute name="VALUE" x="30.353" y="7.503" size="1.27" layer="27" ratio="10" rot="R270"/>
 </element>
-<element name="C2" library="rcl" library_urn="urn:adsk.eagle:library:334" package="C025-024X044" package3d_urn="urn:adsk.eagle:package:23630/1" value="" x="30.48" y="5.725" smashed="yes" rot="R270">
+<element name="C2" library="rcl" library_urn="urn:adsk.eagle:library:334" package="C025-024X044" package3d_urn="urn:adsk.eagle:package:23630/1" value="33pF" x="30.48" y="5.725" smashed="yes" rot="R270">
 <attribute name="NAME" x="35.627" y="7.503" size="1.27" layer="25" ratio="10" rot="R270"/>
 <attribute name="POPULARITY" value="56" x="30.48" y="5.725" size="1.778" layer="27" rot="R270" display="off"/>
@@
 <attribute name="VALUE" x="27.813" y="7.503" size="1.27" layer="27" ratio="10" rot="R270"/>
 </element>
-<element name="C4" library="rcl" library_urn="urn:adsk.eagle:library:334" package="C050-024X044" package3d_urn="urn:adsk.eagle:package:23643/1" value="" x="20.32" y="31.125" smashed="yes">
+<element name="C4" library="rcl" library_urn="urn:adsk.eagle:library:334" package="C050-024X044" package3d_urn="urn:adsk.eagle:package:23643/1" value="100n" x="20.32" y="31.125" smashed="yes">
 <attribute name="NAME" x="14.391" y="30.276" size="1.27" layer="25" ratio="10"/>
 <attribute name="POPULARITY" value="33" x="20.32" y="31.125" size="1.778" layer="27" display="off"/>
@@
 <attribute name="VALUE" x="5.8674" y="26.4006" size="0.9906" layer="27" ratio="10" rot="R270"/>
 </element>
-<element name="C6" library="rcl" library_urn="urn:adsk.eagle:library:334" package="C050-024X044" package3d_urn="urn:adsk.eagle:package:23643/1" value="" x="3.81" y="24.775" smashed="yes" rot="R90">
+<element name="C6" library="rcl" library_urn="urn:adsk.eagle:library:334" package="C050-024X044" package3d_urn="urn:adsk.eagle:package:23643/1" value="100n" x="3.81" y="24.775" smashed="yes" rot="R90">
 <attribute name="NAME" x="2.159" y="21.346" size="1.27" layer="25" ratio="10" rot="R90"/>
 <attribute name="POPULARITY" value="33" x="3.81" y="24.775" size="1.778" layer="27" rot="R90" display="off"/>
@@
 <attribute name="VALUE" x="6.604" y="21.346" size="1.27" layer="27" ratio="10" rot="R90"/>
 </element>
-<element name="C7" library="rcl" library_urn="urn:adsk.eagle:library:334" package="C050-024X044" package3d_urn="urn:adsk.eagle:package:23643/1" value="" x="23.505" y="15.885" smashed="yes" rot="R90">
+<element name="C7" library="rcl" library_urn="urn:adsk.eagle:library:334" package="C050-024X044" package3d_urn="urn:adsk.eagle:package:23643/1" value="100n" x="23.505" y="15.885" smashed="yes" rot="R90">
 <attribute name="NAME" x="22.479" y="17.456" size="1.27" layer="25" ratio="10" rot="R90"/>
 <attribute name="POPULARITY" value="33" x="23.505" y="15.885" size="1.778" layer="27" rot="R90" display="off"/>
