File: Hardware/arduino-nano-dcc-v3.brd (EAGLE design)
At the start: 58.7 x 44.5 mm, 45 parts, among them IC1 7805TV, IC3 MEGA328-P, Q1 16MHz, Q2 TIP41C, X1 22-23-2031

Commit message: Updated hardware t V3, added to pin D7 jumper to enable console mode.
Parts:
- added JP1: (no value), jumper:JP1
Connections:
- new net CONS: IC3.13, JP1.1
- net GND: now also JP1.2
Routing:
- net GND: track 226.9 -> 256.0 mm
- net CONS: track 0.00 -> 29.1 mm, vias 0 -> 1
Other:
- board text added: "DCC SERVO REV 03"
- board text removed: "DCC SERVO REV 02"
Changed lines of the file:
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@@
 <wire x1="0" y1="44.46" x2="0" y2="0" width="0" layer="20"/>
 <text x="28.125" y="22.5" size="1.778" layer="25">DCC SERVO
-REV 02</text>
+REV 03</text>
 </plain>
 <attributes>
@@
 <attribute name="VALUE" x="25.2294" y="12.4424" size="0.9906" layer="27" ratio="10"/>
 </element>
+<element name="JP1" library="jumper" library_urn="urn:adsk.eagle:library:252" package="JP1" package3d_urn="urn:adsk.eagle:package:15455/1" value="" x="48.75" y="5" smashed="yes" rot="R180">
+<attribute name="NAME" x="50.665" y="2.099" size="1.27" layer="25" ratio="10" rot="R180"/>
+<attribute name="POPULARITY" value="61" x="48.75" y="5" size="1.778" layer="27" rot="R180" display="off"/>
+<attribute name="VALUE" x="45.829" y="7.54" size="1.27" layer="27" ratio="10" rot="R270"/>
+</element>
 </elements>
 <signals>
@@
 <wire x1="13.75" y1="8.75" x2="7.5" y2="8.75" width="0.6096" layer="1"/>
 <wire x1="7.5" y1="8.75" x2="7.5" y2="12.075" width="0.6096" layer="1"/>
+<contactref element="JP1" pad="2"/>
+<wire x1="48.75" y1="3.73" x2="46.875" y2="3.73" width="0.6096" layer="16"/>
+<wire x1="46.875" y1="3.73" x2="46.875" y2="3.75" width="0.6096" layer="16"/>
+<wire x1="46.875" y1="3.75" x2="46.875" y2="5.0508" width="0.6096" layer="16"/>
+<wire x1="46.875" y1="5.0508" x2="46.7688" y2="5.0508" width="0.6096" layer="16"/>
+<wire x1="46.7688" y1="5.0508" x2="46.7688" y2="7.4892" width="0.6096" layer="16"/>
+<wire x1="46.7688" y1="7.4892" x2="46.875" y2="7.4892" width="0.6096" layer="16"/>
+<wire x1="56.875" y1="9.375" x2="56.875" y2="17.5" width="0.6096" layer="16"/>
+<wire x1="56.875" y1="17.5" x2="53.965" y2="17.5" width="0.6096" layer="16"/>
+<wire x1="53.965" y1="17.5" x2="53.965" y2="17.115" width="0.6096" layer="16"/>
+<wire x1="46.875" y1="7.4892" x2="46.875" y2="9.375" width="0.6096" layer="16"/>
+<wire x1="46.875" y1="9.375" x2="56.875" y2="9.375" width="0.6096" layer="16"/>
 </signal>
 <signal name="N$17">
@@
 <wire x1="28.145" y1="12.925" x2="28.125" y2="12.925" width="0.4064" layer="1"/>
 </signal>
+<signal name="CONS">
+<contactref element="IC3" pad="13"/>
+<contactref element="JP1" pad="1"/>
+<wire x1="48.75" y1="6.27" x2="48.75" y2="8.75" width="0.6096" layer="1"/>
+<wire x1="48.75" y1="8.75" x2="37.5" y2="8.75" width="0.6096" layer="1"/>
+<wire x1="37.5" y1="8.75" x2="37.5" y2="15.625" width="0.6096" layer="1"/>
+<via x="37.5" y="15.625" extent="1-16" drill="0.35"/>
+<wire x1="37.5" y1="15.625" x2="37.5" y2="19.0854" width="0.6096" layer="16"/>
+<wire x1="37.5" y1="19.0854" x2="39.2684" y2="19.0854" width="0.6096" layer="16"/>
+<wire x1="39.2684" y1="19.0854" x2="39.2684" y2="20.625" width="0.6096" layer="16"/>
+<wire x1="40.64" y1="20.625" x2="40.64" y2="20.965" width="0.6096" layer="16"/>
+<wire x1="39.2684" y1="20.625" x2="40.64" y2="20.625" width="0.6096" layer="16"/>
+</signal>
 </signals>
