File: Hardware/arduino-nano-dcc-v3.sch (EAGLE design)
At the start: 45 parts, among them IC1 7805TV, IC3 MEGA328-P, Q1 16MHz, Q2 TIP41C, X1 22-23-2031

Commit message: Updated hardware t V3, added to pin D7 jumper to enable console mode.
Parts:
- added JP1: (no value), jumper:JP1E
Connections:
- new net CONS: IC3.PD7(AIN1), JP1.1
- net GND: now also JP1.2
Other:
- note added: "3"
- note removed: "2"
Changed lines of the file:
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@@
 <part name="P+2" library="supply1" library_urn="urn:adsk.eagle:library:371" deviceset="+5V" device=""/>
 <part name="R13" library="rcl" deviceset="R-EU_" device="0204/2V" value="10k"/>
+<part name="JP1" library="jumper" library_urn="urn:adsk.eagle:library:252" deviceset="JP1E" device="" package3d_urn="urn:adsk.eagle:package:15455/1"/>
+<part name="GND20" library="supply1" deviceset="GND" device=""/>
 </parts>
 <sheets>
 <sheet>
 <plain>
-<text x="381" y="7.62" size="1.778" layer="91">2</text>
+<text x="381" y="7.62" size="1.778" layer="91">3</text>
 </plain>
 <instances>
@@
 </instance>
 <instance part="R5" gate="G$1" x="170.18" y="241.3" smashed="yes" rot="R180">
-<attribute name="NAME" x="173.99" y="239.8014" size="1.778" layer="95" rot="R180"/>
-<attribute name="VALUE" x="173.99" y="244.602" size="1.778" layer="96" rot="R180"/>
+<attribute name="NAME" x="171.45" y="247.4214" size="1.778" layer="95" rot="R180"/>
+<attribute name="VALUE" x="171.45" y="244.602" size="1.778" layer="96" rot="R180"/>
 </instance>
 <instance part="R6" gate="G$1" x="218.44" y="238.76" smashed="yes" rot="R180">
-<attribute name="NAME" x="222.25" y="237.2614" size="1.778" layer="95" rot="R180"/>
-<attribute name="VALUE" x="222.25" y="242.062" size="1.778" layer="96" rot="R180"/>
+<attribute name="NAME" x="222.25" y="232.1814" size="1.778" layer="95" rot="R180"/>
+<attribute name="VALUE" x="227.33" y="234.442" size="1.778" layer="96" rot="R180"/>
 </instance>
 <instance part="R7" gate="G$1" x="218.44" y="236.22" smashed="yes" rot="R180">
 <attribute name="NAME" x="222.25" y="234.7214" size="1.778" layer="95" rot="R180"/>
-<attribute name="VALUE" x="222.25" y="239.522" size="1.778" layer="96" rot="R180"/>
+<attribute name="VALUE" x="227.33" y="231.902" size="1.778" layer="96" rot="R180"/>
 </instance>
 <instance part="D1" gate="G$1" x="172.72" y="236.22" smashed="yes">
@@
 <attribute name="VALUE" x="231.14" y="256.54" size="1.778" layer="96" rot="R180"/>
 </instance>
-<instance part="SUPPLY1" gate="G$1" x="297.18" y="142.24" smashed="yes" rot="MR270">
-<attribute name="VALUE" x="294.005" y="146.05" size="1.778" layer="96" rot="MR270"/>
+<instance part="SUPPLY1" gate="G$1" x="299.72" y="142.24" smashed="yes" rot="MR270">
+<attribute name="VALUE" x="295.91" y="142.875" size="1.778" layer="96" rot="MR0"/>
 </instance>
 <instance part="SUPPLY2" gate="G$1" x="299.72" y="175.26" smashed="yes" rot="MR270">
-<attribute name="VALUE" x="296.545" y="179.07" size="1.778" layer="96" rot="MR270"/>
+<attribute name="VALUE" x="295.91" y="175.895" size="1.778" layer="96" rot="MR0"/>
 </instance>
 <instance part="SUPPLY3" gate="G$1" x="299.72" y="205.74" smashed="yes" rot="MR270">
-<attribute name="VALUE" x="296.545" y="209.55" size="1.778" layer="96" rot="MR270"/>
+<attribute name="VALUE" x="295.91" y="206.375" size="1.778" layer="96" rot="MR0"/>
 </instance>
 <instance part="SUPPLY4" gate="G$1" x="299.72" y="236.22" smashed="yes" rot="MR270">
-<attribute name="VALUE" x="296.545" y="240.03" size="1.778" layer="96" rot="MR270"/>
+<attribute name="VALUE" x="295.91" y="236.855" size="1.778" layer="96" rot="MR0"/>
 </instance>
 <instance part="SUPPLY5" gate="G$1" x="302.26" y="81.28" smashed="yes" rot="MR270">
-<attribute name="VALUE" x="299.085" y="85.09" size="1.778" layer="96" rot="MR270"/>
+<attribute name="VALUE" x="298.45" y="81.915" size="1.778" layer="96" rot="MR0"/>
 </instance>
 <instance part="SUPPLY6" gate="G$1" x="302.26" y="111.76" smashed="yes" rot="MR270">
-<attribute name="VALUE" x="299.085" y="115.57" size="1.778" layer="96" rot="MR270"/>
+<attribute name="VALUE" x="298.45" y="112.395" size="1.778" layer="96" rot="MR0"/>
 </instance>
 <instance part="SUPPLY10" gate="G$1" x="314.96" y="134.62" smashed="yes" rot="MR270">
@@
 </instance>
 <instance part="R10" gate="G$1" x="134.62" y="91.44" smashed="yes" rot="MR270">
-<attribute name="NAME" x="133.1214" y="95.25" size="1.778" layer="95" rot="MR270"/>
-<attribute name="VALUE" x="137.922" y="95.25" size="1.778" layer="96" rot="MR270"/>
+<attribute name="NAME" x="138.43" y="92.4814" size="1.778" layer="95" rot="MR180"/>
+<attribute name="VALUE" x="138.43" y="89.662" size="1.778" layer="96" rot="MR180"/>
 </instance>
 <instance part="C6" gate="G$1" x="134.62" y="48.26" smashed="yes">
@@
 </instance>
 <instance part="SUPPLY8" gate="G$1" x="246.38" y="167.64" smashed="yes" rot="MR90">
-<attribute name="VALUE" x="249.555" y="163.83" size="1.778" layer="96" rot="MR90"/>
+<attribute name="VALUE" x="250.19" y="169.545" size="1.778" layer="96" rot="MR180"/>
 </instance>
 <instance part="SUPPLY9" gate="G$1" x="233.68" y="157.48" smashed="yes" rot="MR90">
@@
 </instance>
 <instance part="SUPPLY17" gate="G$1" x="246.38" y="139.7" smashed="yes" rot="MR90">
-<attribute name="VALUE" x="249.555" y="135.89" size="1.778" layer="96" rot="MR90"/>
+<attribute name="VALUE" x="250.19" y="141.605" size="1.778" layer="96" rot="MR180"/>
 </instance>
 <instance part="R12" gate="G$1" x="236.22" y="139.7" smashed="yes" rot="MR0">
@@
 <attribute name="VALUE" x="217.17" y="107.442" size="1.778" layer="96" rot="MR180"/>
 </instance>
+<instance part="JP1" gate="A" x="220.98" y="203.2" smashed="yes" rot="R90">
+<attribute name="NAME" x="220.98" y="201.93" size="1.778" layer="95" rot="R180"/>
+<attribute name="VALUE" x="220.98" y="208.915" size="1.778" layer="96" rot="R180"/>
+</instance>
+<instance part="GND20" gate="1" x="228.6" y="205.74" smashed="yes" rot="R90">
+<attribute name="VALUE" x="231.14" y="205.74" size="1.778" layer="96"/>
+</instance>
 </instances>
 <busses>
-<bus name="DCC_IN,LED,RESET,RX,SERVO[1..8],TX">
+<bus name="CONS,DCC_IN,LED,RESET,RX,SERVO[1..8],TX">
 <segment>
 <wire x1="259.08" y1="243.84" x2="259.08" y2="17.78" width="0.762" layer="92"/>
-<label x="261.62" y="205.74" size="1.778" layer="95"/>
+<label x="256.54" y="246.38" size="1.778" layer="95"/>
 </segment>
 </bus>
@@
 <wire x1="228.6" y1="154.94" x2="228.6" y2="152.4" width="0.1524" layer="91"/>
 </segment>
+<segment>
+<pinref part="JP1" gate="A" pin="2"/>
+<pinref part="GND20" gate="1" pin="GND"/>
+<wire x1="226.06" y1="205.74" x2="223.52" y2="205.74" width="0.1524" layer="91"/>
+</segment>
 </net>
 <net name="N$17" class="0">
@@
 <segment>
 <pinref part="R4" gate="G$1" pin="2"/>
-<wire x1="299.72" y1="142.24" x2="304.8" y2="142.24" width="0.1524" layer="91"/>
+<wire x1="302.26" y1="142.24" x2="304.8" y2="142.24" width="0.1524" layer="91"/>
 <pinref part="SUPPLY1" gate="G$1" pin="+5V/2"/>
 </segment>
@@
 </segment>
 </net>
+<net name="CONS" class="0">
+<segment>
+<wire x1="259.08" y1="40.64" x2="256.54" y2="43.18" width="0.1524" layer="91"/>
+<pinref part="IC3" gate="G$1" pin="PD7(AIN1)"/>
+<wire x1="256.54" y1="43.18" x2="233.68" y2="43.18" width="0.1524" layer="91"/>
+<label x="243.84" y="43.18" size="1.778" layer="95"/>
+</segment>
+<segment>
+<wire x1="259.08" y1="200.66" x2="256.54" y2="203.2" width="0.1524" layer="91"/>
+<pinref part="JP1" gate="A" pin="1"/>
+<wire x1="256.54" y1="203.2" x2="223.52" y2="203.2" width="0.1524" layer="91"/>
+</segment>
+</net>
